File: boards/01-power/_restore_backup_2026-07-01T13-46-12-633/power.kicad_pcb (KiCad board)
At the start: 6 copper layers, 50 x 50 mm, 42 parts, among them J1 CONN_DF40_100P_F, J2 USB_C_Receptacle_USB2.0_16P, J3 TC2030, P1 MAG_RB1_125BAG1A, U1 USBLC6-2P6, U2 AP63203WU, U3 STM32F405RGTx, Y1 16Mhz

Commit message: chore: layout
Parts:
- moved U1 75.7 mm to (88.0, 88.2), turned to 90 degrees
- moved F1 74.5 mm to (84.0, 88.2), turned to 90 degrees
- moved R1 71.7 mm to (86.0, 88.2), turned to 90 degrees
- moved R2 67.1 mm to (90.0, 88.2), turned to 90 degrees
- moved J3 63.8 mm to (75.0, 66.0), turned to -90 degrees
- moved U3 56.9 mm to (90.6, 78.2), turned to -90 degrees
- moved Y1 54.9 mm to (91.1, 67.2), turned to 180 degrees
- moved C17 42.4 mm to (87.8, 67.3), turned to 90 degrees
- moved C16 37.2 mm to (94.3, 67.2), turned to -90 degrees
- moved R5 37.1 mm to (97.8, 60.5), turned to 180 degrees
- moved R6 35.1 mm to (97.8, 56.5), turned to 180 degrees
- moved D2 27.4 mm to (97.8, 58.5), turned to 180 degrees
- moved D1 26.3 mm to (97.8, 62.5), turned to 180 degrees
Connections:
- D1 pad 1: GND -> Net-(D1-K)
- D1 pad 2: Net-(D1-A) -> /STM32/LED_STATUS
- D2 pad 1: GND -> Net-(D2-K)
- D2 pad 2: Net-(D2-A) -> /STM32/LED_ERROR
- R5 pad 1: /STM32/LED_STATUS -> Net-(D1-K)
- R5 pad 2: Net-(D1-A) -> GND
- R6 pad 1: /STM32/LED_ERROR -> Net-(D2-K)
- R6 pad 2: Net-(D2-A) -> GND

Commit message: chore: layout pours
Parts:
- moved U2 83.6 mm to (82.6, 85.5)
- moved C2 83.2 mm to (79.8, 89.2), turned to -90 degrees
- moved C1 82.9 mm to (81.5, 89.2), turned to -90 degrees
- moved L1 79.9 mm to (82.6, 81.6), turned to 180 degrees
- moved C3 79.9 mm to (79.0, 82.5), turned to 180 degrees
- moved C4 78.3 mm to (79.0, 80.7), turned to 180 degrees
- moved R3 75.2 mm to (79.8, 85.5), turned to 90 degrees
- moved C5 73.1 mm to (85.5, 85.5), turned to 90 degrees
- moved J3 26.0 mm to (95.5, 82.0), turned to 180 degrees
- moved U3 10.8 mm to (89.0, 67.5)
- moved C16 9.65 mm to (94.2, 57.5)
- moved Y1 9.65 mm to (91.0, 57.5)
- moved C17 9.65 mm to (87.8, 57.6)
- moved P1 1.50 mm to (64.5, 89.0)
- moved R1 1.40 mm to (85.0, 89.2)
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Routing:
- net /USB/~{EN}: track 0.00 -> 2.08 mm
- net Net-(U2-SW): track 0.00 -> 2.06 mm
- added copper zone on F.Cu, net /USB/+3.3V
- added copper zone on F.Cu, net /USB/VBUS
- added copper zone on F.Cu, net Net-(U2-BST)
