File: boards/01-power/power.kicad_pcb (KiCad board)
At the start: 6 copper layers, 50 x 50 mm, 7 parts, among them J1 CONN_DF40_100P_F, J2 CONN_USB_C_M, P1 MAG_RB1_125BAG1A

Commit message: chore: usb/stm32 schematic
Parts:
- added C1: 22uF, Capacitor_SMD:C_0603_1608Metric, F.Cu at (156.0, 51.3)
- added C10: 100nF, Capacitor_SMD:C_0603_1608Metric, F.Cu at (127.5, 58.8)
- added C11: 100nF, Capacitor_SMD:C_0603_1608Metric, F.Cu at (127.5, 61.3)
- added C12: 100nF, Capacitor_SMD:C_0603_1608Metric, F.Cu at (127.5, 63.8)
- added C13: 100nF, Capacitor_SMD:C_0603_1608Metric, F.Cu at (127.5, 66.3)
- added C14: 100nF, Capacitor_SMD:C_0603_1608Metric, F.Cu at (131.5, 51.3)
- added C15: 100nF, Capacitor_SMD:C_0603_1608Metric, F.Cu at (131.5, 53.8)
- added C16: 30pF, Capacitor_SMD:C_0603_1608Metric, F.Cu at (131.5, 56.3)
- added C17: 30pF, Capacitor_SMD:C_0603_1608Metric, F.Cu at (131.5, 58.8)
- added C18: 100nF, Capacitor_SMD:C_0603_1608Metric, F.Cu at (131.5, 61.3)
- added C2: 100nF, Capacitor_SMD:C_0603_1608Metric, F.Cu at (156.0, 53.8)
- added C3: 22uF, Capacitor_SMD:C_0603_1608Metric, F.Cu at (156.0, 56.3)
- added C4: 22uF, Capacitor_SMD:C_0603_1608Metric, F.Cu at (156.0, 58.8)
- added C5: 100nF, Capacitor_SMD:C_0603_1608Metric, F.Cu at (156.0, 61.3)
- added C6: 2.2uF, Capacitor_SMD:C_0603_1608Metric, F.Cu at (127.5, 51.3)
- added C7: 2.2uF, Capacitor_SMD:C_0603_1608Metric, F.Cu at (127.5, 53.8)
- added C8: 2.2uF, Capacitor_SMD:C_0603_1608Metric, F.Cu at (127.5, 56.3)
- added D1: ST, LED_SMD:LED_0603_1608Metric, F.Cu at (145.8, 70.3)
- added D2: ST, LED_SMD:LED_0603_1608Metric, F.Cu at (145.8, 72.9)
- added F1: Polyfuse, Fuse:Fuse_0603_1608Metric, F.Cu at (156.0, 63.8)
- added FB1: FB, Inductor_SMD:L_0603_1608Metric, F.Cu at (131.5, 63.8)
- added L1: L_Small, Inductor_SMD:L_APV_ANR3012, F.Cu at (160.3, 56.9)
- added R1: 5.1k, Resistor_SMD:R_0603_1608Metric, F.Cu at (156.0, 66.3)
- added R2: 5.1k, Resistor_SMD:R_0603_1608Metric, F.Cu at (156.0, 68.8)
- added R3: 10k, Resistor_SMD:R_0603_1608Metric, F.Cu at (156.0, 71.3)
- added R4: 10k, Resistor_SMD:R_0603_1608Metric, F.Cu at (131.5, 66.3)
- added R5: 300R, Resistor_SMD:R_0603_1608Metric, F.Cu at (135.5, 51.3)
- added R6: 300R, Resistor_SMD:R_0603_1608Metric, F.Cu at (135.5, 53.8)
- added R7: 10k, Resistor_SMD:R_0603_1608Metric, F.Cu at (135.5, 56.3)
- added R8: 10k, Resistor_SMD:R_0603_1608Metric, F.Cu at (135.5, 58.8)
- added SW1: SW_BOOT, Woki:SW_B3U_1000P, F.Cu at (140.9, 66.5)
- added SW2: SW_BOOT, Woki:SW_B3U_1000P, F.Cu at (140.9, 70.5)
- added SW3: SW_BOOT, Woki:SW_B3U_1000P, F.Cu at (140.9, 74.6)
- added U1: USBLC6-2P6, Package_TO_SOT_SMD:SOT-666, F.Cu at (126.5, 76.0)
- added U2: AP63203WU, Package_TO_SOT_SMD:TSOT-23-6, F.Cu at (160.6, 52.4)
- added U3: STM32F405RGTx, Package_QFP:LQFP-64_10x10mm_P0.5mm, F.Cu at (144.8, 57.2)
- added Y1: 16Mhz, Crystal:Crystal_SMD_3225-4Pin_3.2x2.5mm, F.Cu at (146.4, 66.7)
- J2: value CONN_USB_C_M -> USB_C_Receptacle_USB2.0_16P
Connections:
- J1 pad 1: (no net) -> +12V_BULK
- J1 pad 10: (no net) -> +12V_BULK
- J1 pad 100: (no net) -> GND
- J1 pad 11: (no net) -> +12V_BULK
- J1 pad 12: (no net) -> +12V_BULK
- J1 pad 13: (no net) -> +12V_BULK
- J1 pad 14: (no net) -> +12V_BULK
- J1 pad 15: (no net) -> +12V_BULK
- J1 pad 16: (no net) -> +12V_BULK
- J1 pad 17: (no net) -> GND
- J1 pad 18: (no net) -> GND
- J1 pad 19: (no net) -> GND
- J1 pad 2: (no net) -> +12V_BULK
- J1 pad 20: (no net) -> GND
- J1 pad 21: (no net) -> GND
- J1 pad 22: (no net) -> GND
- J1 pad 23: (no net) -> GND
- J1 pad 24: (no net) -> GND
- J1 pad 25: (no net) -> GND
- J1 pad 26: (no net) -> GND
- J1 pad 27: (no net) -> GND
- J1 pad 28: (no net) -> GND
- J1 pad 29: (no net) -> +5V_AUX
- J1 pad 3: (no net) -> +12V_BULK
- J1 pad 30: (no net) -> +5V_AUX
- J1 pad 31: (no net) -> +5V_AUX
- J1 pad 32: (no net) -> +5V_AUX
- J1 pad 33: (no net) -> +3V3_STBY
- J1 pad 34: (no net) -> +3V3_STBY
- J1 pad 35: (no net) -> GND
- J1 pad 36: (no net) -> GND
- J1 pad 37: (no net) -> GND
- J1 pad 38: (no net) -> GND
- J1 pad 39: (no net) -> /FPGA_JTAG_TCK
- J1 pad 4: (no net) -> +12V_BULK
- J1 pad 40: (no net) -> /FPGA_JTAG_TMS
- J1 pad 41: (no net) -> /FPGA_JTAG_TDI
- J1 pad 42: (no net) -> /FPGA_JTAG_TDO
- J1 pad 43: (no net) -> /FPGA_JTAG_VREF
- J1 pad 44: (no net) -> /FPGA_DEBUG_RESET_N
- J1 pad 45: (no net) -> GND
- J1 pad 46: (no net) -> GND
- J1 pad 47: (no net) -> /STM_SWDIO
- J1 pad 48: (no net) -> /STM_SWCLK
- J1 pad 49: (no net) -> /STM_NRST
- J1 pad 5: (no net) -> +12V_BULK
- J1 pad 50: (no net) -> /STM_SWO
- J1 pad 51: (no net) -> /STM_VREF
- J1 pad 52: (no net) -> GND
- J1 pad 53: (no net) -> GND
- J1 pad 54: (no net) -> /FPGA_PROGRAM_B
- J1 pad 55: (no net) -> /FPGA_INIT_B
- J1 pad 56: (no net) -> /FPGA_DONE
- J1 pad 57: (no net) -> /FPGA_CFG_CLK
- J1 pad 58: (no net) -> /FPGA_CFG_DATA
- J1 pad 59: (no net) -> GND
- J1 pad 6: (no net) -> +12V_BULK
- J1 pad 60: (no net) -> GND
- J1 pad 61: (no net) -> /RGMII_TXC
- J1 pad 62: (no net) -> /RGMII_TX_CTL
- J1 pad 63: (no net) -> /RGMII_TXD0
- J1 pad 64: (no net) -> /RGMII_TXD1
- J1 pad 65: (no net) -> /RGMII_TXD2
- J1 pad 66: (no net) -> /RGMII_TXD3
- J1 pad 67: (no net) -> /RGMII_TX_SPARE
- J1 pad 68: (no net) -> GND
- J1 pad 69: (no net) -> GND
- J1 pad 7: (no net) -> +12V_BULK
- J1 pad 70: (no net) -> /RGMII_RXC
- J1 pad 71: (no net) -> /RGMII_RX_CTL
- J1 pad 72: (no net) -> /RGMII_RXD0
- J1 pad 73: (no net) -> /RGMII_RXD1
- J1 pad 74: (no net) -> /RGMII_RXD2
- J1 pad 75: (no net) -> /RGMII_RXD3
- J1 pad 76: (no net) -> /RGMII_RX_SPARE
- J1 pad 77: (no net) -> GND
- J1 pad 78: (no net) -> GND
- J1 pad 79: (no net) -> /ETH_MDC
- J1 pad 8: (no net) -> +12V_BULK
- J1 pad 80: (no net) -> /ETH_MDIO
- J1 pad 81: (no net) -> /ETH_PHY_RESET_N
- J1 pad 82: (no net) -> /ETH_PHY_INT_N
- J1 pad 83: (no net) -> /ETH_REFCLK_125M
- J1 pad 84: (no net) -> /ETH_CLK_ENABLE
- J1 pad 85: (no net) -> GND
- J1 pad 86: (no net) -> GND
- J1 pad 87: (no net) -> /STACK_I2C_SCL
- J1 pad 88: (no net) -> /STACK_I2C_SDA
- J1 pad 89: (no net) -> /STACK_SYNC_OUT
- J1 pad 9: (no net) -> +12V_BULK
- J1 pad 90: (no net) -> /STACK_SYNC_IN
- J1 pad 91: (no net) -> /STACK_CAM_TRIGGER
- J1 pad 92: (no net) -> /STACK_LED_TRIGGER
- J1 pad 93: (no net) -> /STACK_FAULT_N
- J1 pad 94: (no net) -> /STACK_RESET_N
- J1 pad 95: (no net) -> /FPGA_DEBUG0
- J1 pad 96: (no net) -> /FPGA_DEBUG1
- J1 pad 97: (no net) -> /FPGA_DEBUG2
- J1 pad 98: (no net) -> /FPGA_DEBUG3
- J1 pad 99: (no net) -> GND
- J2 pad A1: Net-(J2-GND-PadA1) -> GND
- J2 pad A12: Net-(J2-GND-PadA1) -> GND
- J2 pad A5: unconnected-(J2-CC1-PadA5) -> Net-(J2-CC1)
- J2 pad A6: unconnected-(J2-D+-PadA6) -> /USB/D+
- J2 pad A7: unconnected-(J2-D--PadA7) -> /USB/D-
- J2 pad B1: Net-(J2-GND-PadA1) -> GND
- J2 pad B12: Net-(J2-GND-PadA1) -> GND
- J2 pad B5: unconnected-(J2-CC2-PadB5) -> Net-(J2-CC2)
- J2 pad B6: unconnected-(J2-D+-PadB6) -> /USB/D+
- J2 pad B7: unconnected-(J2-D--PadB7) -> /USB/D-
- J2 pad SH: unconnected-(J2-SHIELD-PadSH) -> GND

Commit message: wip: layout
Parts:
- C1, C2, C3, C4, F1, L1, R1, R2, R3, U1, U2: moved to B.Cu
- moved R1 80.0 mm to (79.3, 89.0), turned to 90 degrees
- moved U2 78.2 mm to (91.5, 89.0)
- moved C3 77.8 mm to (89.5, 96.8)
- moved L1 77.7 mm to (91.5, 93.0), turned to 180 degrees
- moved C4 77.6 mm to (89.5, 98.8)
- moved C2 77.0 mm to (85.8, 85.2), turned to 90 degrees
- moved C1 76.2 mm to (87.8, 85.2), turned to 90 degrees
- moved R2 74.8 mm to (83.9, 89.0), turned to 90 degrees
- moved F1 74.6 mm to (85.8, 89.0), turned to 90 degrees
- moved R3 70.5 mm to (87.8, 89.0), turned to -90 degrees
- moved U3 61.7 mm to (86.5, 77.6), turned to 180 degrees
- moved U1 46.8 mm to (81.5, 89.0), turned to 90 degrees
- moved J2 6.25 mm to (81.9, 96.3)
- moved P1 0.50 mm to (65.5, 89.0)
Routing:
- net +12V_BULK: track 0.00 -> 1.54 mm, vias 0 -> 1
- added copper zone on In3.Cu, net +12V_BULK
- added copper zone on In1.Cu, net GND
- added copper zone on In4.Cu, net GND

Commit message: wip: 8 layer stackup
Connections:
- C10 pad 1: /STM32/+3.3V -> +3.3V
- C11 pad 1: /STM32/+3.3V -> +3.3V
- C12 pad 1: /STM32/+3.3V -> +3.3V
- C13 pad 1: /STM32/+3.3V -> +3.3V
- C14 pad 1: /STM32/+3.3V -> +3.3V
- C15 pad 1: /STM32/+3.3V -> +3.3V
- C3 pad 1: /USB/+3.3V -> +3.3V
- C4 pad 1: /USB/+3.3V -> +3.3V
- C6 pad 1: /STM32/+3.3V -> +3.3V
- FB1 pad 1: /STM32/+3.3V -> +3.3V
- L1 pad 2: /USB/+3.3V -> +3.3V
- SW1 pad 2: /STM32/+3.3V -> +3.3V
- SW2 pad 2: /STM32/+3.3V -> +3.3V
- SW3 pad 2: /STM32/+3.3V -> +3.3V
- U2 pad 1: /USB/+3.3V -> +3.3V
- U3 pad 1: /STM32/+3.3V -> +3.3V
- U3 pad 19: /STM32/+3.3V -> +3.3V
- U3 pad 32: /STM32/+3.3V -> +3.3V
- U3 pad 48: /STM32/+3.3V -> +3.3V
- U3 pad 64: /STM32/+3.3V -> +3.3V
Routing:
- net +3.3V: vias 0 -> 4
- added copper zone on In5.Cu, net +3.3V
Other:
- copper layers 6 -> 8
Changed lines of the file:
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@@
 		(8 "In3.Cu" power "PWR")
 		(10 "In4.Cu" power "GND2")
+		(12 "In5.Cu" power "+3.3V")
+		(14 "In6.Cu" power "GND3")
 		(2 "B.Cu" signal)
 		(5 "F.SilkS" user "F.Silkscreen")
@@
 				(type "core")
 				(color "#FF9B30FF")
-				(thickness 0.545)
+				(thickness 0.18)
 				(material "FR4")
 				(epsilon_r 4.5)
@@
 				(type "core")
 				(color "#FF7030FF")
-				(thickness 0.545)
+				(thickness 0.56)
 				(material "FR4")
 				(epsilon_r 4.5)
@@
 				(loss_tangent 0.02)
 			)
+			(layer "In5.Cu"
+				(type "copper")
+				(thickness 0.035)
+			)
+			(layer "dielectric 6"
+				(type "core")
+				(color "#FF9B30FF")
+				(thickness 0.18)
+				(material "FR4")
+				(epsilon_r 4.5)
+				(loss_tangent 0.02)
+			)
+			(layer "In6.Cu"
+				(type "copper")
+				(thickness 0.035)
+			)
+			(layer "dielectric 7"
+				(type "prepreg")
+				(color "#30FF19FF")
+				(thickness 0.1)
+				(material "FR4")
+				(epsilon_r 4.5)
+				(loss_tangent 0.02)
+			)
 			(layer "B.Cu"
 				(type "copper")
@@
 			(layers "F.Cu" "F.Mask" "F.Paste")
 			(roundrect_rratio 0.25)
-			(net "/STM32/+3.3V")
+			(net "+3.3V")
 			(pintype "passive")
 		)
@@
 			(layers "F.Cu" "F.Mask" "F.Paste")
 			(roundrect_rratio 0.25)
-			(net "/STM32/+3.3V")
+			(net "+3.3V")
 			(pintype "passive")
 		)
@@
 			(size 0.8 1.7)
 			(layers "F.Cu" "F.Mask" "F.Paste")
-			(net "/STM32/+3.3V")
+			(net "+3.3V")
 			(pinfunction "2_2")
 			(pintype "passive")
@@
 			(layers "F.Cu" "F.Mask" "F.Paste")
 			(roundrect_rratio 0.25)
-			(net "/STM32/+3.3V")
+			(net "+3.3V")
 			(pintype "passive")
 		)
@@
 			(layers "F.Cu" "F.Mask" "F.Paste")
 			(roundrect_rratio 0.25)
-			(net "/STM32/+3.3V")
+			(net "+3.3V")
 			(pintype "passive")
 		)
@@
 			(size 0.8 1.7)
 			(layers "F.Cu" "F.Mask" "F.Paste")
-			(net "/STM32/+3.3V")
+			(net "+3.3V")
 			(pinfunction "2_2")
 			(pintype "passive")
@@
 			(layers "F.Cu" "F.Mask" "F.Paste")
 			(roundrect_rratio 0.25)
-			(net "/STM32/+3.3V")
+			(net "+3.3V")
 			(pinfunction "VBAT_1")
 			(pintype "power_in")
@@
 			(layers "F.Cu" "F.Mask" "F.Paste")
 			(roundrect_rratio 0.25)
-			(net "/STM32/+3.3V")
+			(net "+3.3V")
 			(pinfunction "VDD_19")
 			(pintype "power_in")
@@
 			(layers "F.Cu" "F.Mask" "F.Paste")
 			(roundrect_rratio 0.25)
-			(net "/STM32/+3.3V")
+			(net "+3.3V")
 			(pinfunction "VDD_32")
 			(pintype "power_in")
@@
 			(layers "F.Cu" "F.Mask" "F.Paste")
 			(roundrect_rratio 0.25)
-			(net "/STM32/+3.3V")
+			(net "+3.3V")
 			(pinfunction "VDD_48")
 			(pintype "power_in")
@@
 			(layers "F.Cu" "F.Mask" "F.Paste")
 			(roundrect_rratio 0.25)
-			(net "/STM32/+3.3V")
+			(net "+3.3V")
 			(pinfunction "VDD_64")
 			(pintype "power_in")
@@
 			(layers "F.Cu" "F.Mask" "F.Paste")
 			(roundrect_rratio 0.25)
-			(net "/STM32/+3.3V")
+			(net "+3.3V")
 			(pintype "passive")
 		)
@@
 			(layers "F.Cu" "F.Mask" "F.Paste")
 			(roundrect_rratio 0.25)
-			(net "/STM32/+3.3V")
+			(net "+3.3V")
 			(pintype "passive")
 		)
@@
 			(size 0.8 1.7)
 			(layers "F.Cu" "F.Mask" "F.Paste")
-			(net "/STM32/+3.3V")
+			(net "+3.3V")
 			(pinfunction "2_2")
 			(pintype "passive")
@@
 			(layers "F.Cu" "F.Mask" "F.Paste")
 			(roundrect_rratio 0.25)
-			(net "/STM32/+3.3V")
+			(net "+3.3V")
 			(pintype "passive")
 		)
@@
 			(layers "F.Cu" "F.Mask" "F.Paste")
 			(roundrect_rratio 0.25)
-			(net "/STM32/+3.3V")
+			(net "+3.3V")
 			(pintype "passive")
 		)
@@
 			(layers "B.Cu" "B.Mask" "B.Paste")
 			(roundrect_rratio 0.25)
-			(net "/USB/+3.3V")
+			(net "+3.3V")
 			(pinfunction "FB_1")
 			(pintype "input")
@@
 			(layers "B.Cu" "B.Mask" "B.Paste")
 			(roundrect_rratio 0.25)
-			(net "/USB/+3.3V")
+			(net "+3.3V")
 			(pintype "passive")
 		)
@@
 			(layers "B.Cu" "B.Mask" "B.Paste")
 			(roundrect_rratio 0.25)
-			(net "/USB/+3.3V")
+			(net "+3.3V")
 			(pintype "passive")
 		)
@@
 			(layers "B.Cu" "B.Mask" "B.Paste")
 			(roundrect_rratio 0.25)
-			(net "/USB/+3.3V")
+			(net "+3.3V")
 			(pintype "passive")
 		)
@@
 		(layer "Edge.Cuts")
 	)
+	(via
+		(at 90.35 93)
+		(size 0.55)
+		(drill 0.25)
+		(layers "F.Cu" "B.Cu")
+		(net "+3.3V")
+	)
+	(via
+		(at 90.3625 89.95)
+		(size 0.55)
+		(drill 0.25)
+		(layers "F.Cu" "B.Cu")
+		(net "+3.3V")
+	)
+	(via
+		(at 88.725 98.75)
+		(size 0.55)
+		(drill 0.25)
+		(layers "F.Cu" "B.Cu")
+		(net "+3.3V")
+	)
+	(via
+		(at 88.725 96.75)
+		(size 0.55)
+		(drill 0.25)
+		(layers "F.Cu" "B.Cu")
+		(net "+3.3V")
+	)
 	(segment
 		(start 84.8 53.6096)
@@
 		(hatch edge 0.5)
 		(connect_pads
+			(clearance 0.2)
+		)
+		(min_thickness 0.127)
+		(fill yes
+			(thermal_gap 0.2)
+			(thermal_bridge_width 0.25)
+			(island_removal_mode 0)
+		)
+		(polygon
+			(pts
+				(xy 53 50) (xy 97 50) (xy 97.391579 50.025665) (xy 97.776457 50.102223) (xy 98.14805 50.228361)
+				(xy 98.5 50.401924) (xy 98.826284 50.61994) (xy 99.12132 50.87868) (xy 99.38006 51.173716) (xy 99.598076 51.5)
+				(xy 99.771639 51.85195) (xy 99.897777 52.223543) (xy 99.974335 52.608421) (xy 100 53) (xy 100 97)
+				(xy 99.974335 97.391579) (xy 99.897777 97.776457) (xy 99.771639 98.14805) (xy 99.598076 98.5) (xy 99.38006 98.826284)
+				(xy 99.12132 99.12132) (xy 98.826284 99.38006) (xy 98.5 99.598076) (xy 98.14805 99.771639) (xy 97.776457 99.897777)
+				(xy 97.391579 99.974335) (xy 97 100) (xy 53 100) (xy 52.608421 99.974335) (xy 52.223543 99.897777)
+				(xy 51.85195 99.771639) (xy 51.5 99.598076) (xy 51.173716 99.38006) (xy 50.87868 99.12132) (xy 50.61994 98.826284)
+				(xy 50.401924 98.5) (xy 50.228361 98.14805) (xy 50.102223 97.776457) (xy 50.025665 97.391579) (xy 50 97)
+				(xy 50 53) (xy 50.025665 52.608421) (xy 50.102223 52.223543) (xy 50.228361 51.85195) (xy 50.401924 51.5)
+				(xy 50.61994 51.173716) (xy 50.87868 50.87868) (xy 51.173716 50.61994) (xy 51.5 50.401924) (xy 51.85195 50.228361)
+				(xy 52.223543 50.102223) (xy 52.608421 50.025665)
+			)
+		)
+	)
+	(zone
+		(net "+3.3V")
+		(layer "In5.Cu")
+		(hatch edge 0.5)
+		(connect_pads
