File: boards/01-power/power.kicad_pcb (KiCad board)
At the start: 8 copper layers, 50 x 50 mm, 44 parts, among them J1 CONN_DF40_100P_F, J2 USB_C_Receptacle_USB2.0_16P, P1 MAG_RB1_125BAG1A, SW1 SW_BOOT, SW2 SW_BOOT, SW3 SW_BOOT, U1 USBLC6-2P6, U2 AP63203WU, U3 STM32F405RGTx, Y1 16Mhz

Commit message: wip: 3.3v
Parts:
- removed SW1: SW_BOOT, Woki:SW_B3U_1000P
- added BOOT: SW_BOOT, Woki:SW_B3U_1000P, B.Cu at (95.5, 84.2)
- added J3: TC2030, Connector:Tag-Connect_TC2030-IDC-FP_2x03_P1.27mm_Vertical, F.Cu at (160.6, 81.7)
- added U4: PMIC_TPS2372_4RGWR, Woki:PMIC_TPS2372_4RGWR, F.Cu at (57.8, 70.8)
- C5, D1, D2, R5, R6, SW2, SW3: moved to B.Cu
- moved C5 79.3 mm to (79.0, 80.5)
- moved R6 63.2 mm to (90.5, 98.2), turned to 90 degrees
- moved R5 62.5 mm to (94.2, 98.2), turned to 90 degrees
- moved D2 62.5 mm to (88.7, 98.2), turned to 90 degrees
- moved D1 60.3 mm to (92.4, 98.2), turned to 90 degrees
- moved Y1 53.7 mm to (92.9, 63.2), turned to 180 degrees
- moved SW2 48.8 mm to (95.5, 88.3), turned to 180 degrees
- moved SW3 48.8 mm to (95.5, 92.3), turned to 180 degrees
- moved C17 42.0 mm to (89.8, 63.2), turned to 90 degrees
- moved C16 36.2 mm to (96.0, 63.2), turned to -90 degrees
- moved C12 23.5 mm to (145.8, 78.6)
- moved C8 23.5 mm to (145.8, 71.0)
- moved FB1 23.5 mm to (149.8, 78.6)
- moved R7 23.5 mm to (153.8, 71.0)
- moved C10 23.5 mm to (145.8, 73.5)
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Connections:
- net Net-(U3-NRST) renamed /STM32/~{STM_RESET}
- D1 pad 1: GND -> Net-(D1-K)
- D1 pad 2: Net-(D1-A) -> /STM32/LED_STATUS
- D2 pad 1: GND -> Net-(D2-K)
- D2 pad 2: Net-(D2-A) -> /STM32/LED_ERROR
- R5 pad 1: /STM32/LED_STATUS -> Net-(D1-K)
- R5 pad 2: Net-(D1-A) -> GND
- R6 pad 1: /STM32/LED_ERROR -> Net-(D2-K)
- R6 pad 2: Net-(D2-A) -> GND
Routing:
- net /USB/D-: track 0.00 -> 5.22 mm
- net Net-(U1-VBUS): track 0.00 -> 2.96 mm
- net /USB/D+: track 0.00 -> 2.78 mm
- net /USB/~{EN}: track 0.00 -> 2.32 mm
- net +12V_BULK: track 1.54 -> 0.00 mm, vias 1 -> 0
- net /STM32/USB_D-: track 0.00 -> 1.50 mm, vias 0 -> 1
- net /STM32/USB_D+: track 0.00 -> 1.50 mm, vias 0 -> 1
- net GND: track 0.00 -> 0.67 mm, vias 0 -> 1
- added copper zone on B.Cu, net /USB/VBUS

Commit message: wip: buck (plan layout rough)
Parts:
- removed BOOT, SW3: SW_BOOT, Woki:SW_B3U_1000P
- added SW1: SW_BOOT, Woki:SW_B3U_1000P, B.Cu at (97.0, 60.8)
- U3: moved to B.Cu
- moved J3 106.2 mm to (56.6, 60.3)
- moved FB1 62.1 mm to (87.7, 75.4), turned to 90 degrees
- moved C15 60.4 mm to (89.8, 75.6), turned to 90 degrees
- moved C12 57.9 mm to (87.9, 78.9), turned to 90 degrees
- moved C13 57.5 mm to (88.8, 73.1), turned to 180 degrees
- moved C14 55.9 mm to (94.3, 72.9), turned to 180 degrees
- moved C11 55.5 mm to (90.4, 80.2)
- moved C10 50.9 mm to (95.1, 78.8), turned to 90 degrees
- moved R7 47.3 mm to (108.0, 83.0)
- moved R8 47.3 mm to (108.0, 85.5)
- moved R4 47.3 mm to (104.0, 93.0)
- moved C18 38.5 mm to (111.4, 72.4)
- moved C6 38.5 mm to (107.4, 62.4)
- moved C7 38.5 mm to (107.4, 64.9)
- moved C8 38.5 mm to (107.4, 67.4)
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Connections:
- U3 pad 11: /STM32/USR_BTN2 -> unconnected-(U3-PC3-Pad11)
Routing:
- net Net-(U1-VBUS): track 2.96 -> 14.8 mm
- net GND: track 0.67 -> 9.14 mm, vias 1 -> 7
- net Net-(U2-BST): track 0.00 -> 4.78 mm
- net Net-(U2-SW): track 0.00 -> 4.29 mm
- net Net-(J2-CC1): track 0.00 -> 3.19 mm
- net /USB/D+: track 2.78 -> 5.93 mm, vias 0 -> 2
- net Net-(J2-CC2): track 0.00 -> 2.52 mm
- net /STM32/USB_D-: track 1.50 -> 0.00 mm, vias 1 -> 0
- net /STM32/USB_D+: track 1.50 -> 0.00 mm, vias 1 -> 0
- net +3.3V: vias 0 -> 3
- added copper zone on B.Cu, net +3.3V
- added copper zone on B.Cu, net GND

Commit message: wip: stm
Parts:
- removed R8: 10k, Resistor_SMD:R_0603_1608Metric
- added J4: TC2030, Connector:Tag-Connect_TC2030-IDC-FP_2x03_P1.27mm_Vertical, B.Cu at (57.1, 57.4)
- C10, C11, C12, C13, C14, C15, C8, FB1, J3: moved to B.Cu
- moved U4 62.2 mm to (118.5, 57.0)
- moved C16 53.9 mm to (147.2, 76.3)
- moved C17 53.9 mm to (140.9, 76.3)
- moved Y1 53.9 mm to (144.1, 76.3)
- moved SW1 40.8 mm to (137.2, 54.0)
- moved SW2 40.8 mm to (137.2, 50.8)
- moved J3 36.4 mm to (92.9, 57.4), turned to -135 degrees
- moved C8 27.4 mm to (82.2, 78.3), turned to -90 degrees
- moved C7 27.1 mm to (122.7, 87.3), turned to -90 degrees
- moved C18 17.7 mm to (129.1, 73.4)
- moved R4 17.7 mm to (121.7, 93.9)
- moved C6 17.7 mm to (125.1, 63.3)
- moved R7 17.7 mm to (125.7, 83.9)
- moved C14 16.0 mm to (87.5, 87.4), turned to 0 degrees
- moved C13 14.8 mm to (92.7, 87.4), turned to 0 degrees
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Connections:
- U3 pad 2: /STM32/LED_STATUS -> unconnected-(U3-PC13-Pad2)
- U3 pad 24: unconnected-(U3-PC4-Pad24) -> /STM32/LED_STATUS
- U3 pad 25: unconnected-(U3-PC5-Pad25) -> /STM32/LED_ERROR
- U3 pad 3: /STM32/LED_ERROR -> unconnected-(U3-PC14-Pad3)
Routing:
- net +3.3V: track 0.00 -> 22.6 mm, vias 3 -> 9
- net GND: track 9.14 -> 28.0 mm, vias 7 -> 17
- net /STM32/USB_D+: track 0.00 -> 13.7 mm
- net /STM32/USB_D-: track 0.00 -> 13.0 mm
- net /STM32/LED_STATUS: track 0.00 -> 12.9 mm
- net /STM32/LED_ERROR: track 0.00 -> 12.3 mm
- net Net-(U3-VCAP_2): track 0.00 -> 2.84 mm
- net Net-(D2-K): track 0.00 -> 2.05 mm
- net Net-(D1-K): track 0.00 -> 1.87 mm

Commit message: feat: jtag connector/programer
Parts:
- added JTAG: CONN_TC2030_JTAG, Woki:CONN_TC2030_JTAG_PROBE, F.Cu at (42.0, 66.4)

Commit message: feat: jtag connector/programer
Parts:
- moved JTAG 18.3 mm to (60.1, 69.0), turned to 90 degrees
Changed lines of the file:
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@@
 	(footprint "Woki:CONN_TC2030_JTAG_PROBE"
 		(layer "F.Cu")
-		(at 41.95 66.4)
+		(at 60.08 68.974 90)
 		(descr "Generated from CONN_TC2030_JTAG.kicad_mod; TC2030 pitch 1.27 mm, C5157236 tip 0.80 mm leaves 0.47 mm between tips, barrel 1.20 mm leaves 0.07 mm between barrels")
 		(tags "tc2030 jtag swd pogo probe card-edge")
 		(property "Reference" "JTAG"
-			(at 0 -4.35 180)
+			(at 0 6.875 90)
 			(layer "F.SilkS")
 			(effects
@@
 		)
 		(property "Datasheet" "https://www.tag-connect.com/wp-content/uploads/bsk-pdf-manager/TC2030-CTX_1.pdf"
-			(at 0 0 0)
+			(at 0 0 90)
 			(layer "F.Fab")
 			(hide yes)
@@
 		)
 		(property "Description" "Tag-Connect ARM Cortex SWD JTAG connector, 6 pin"
-			(at 0 0 0)
+			(at 0 0 90)
 			(layer "F.Fab")
 			(hide yes)
@@
 		)
 		(property "Value" "CONN_TC2030_JTAG"
-			(at 0 20 0)
+			(at 0 20 90)
 			(layer "F.Fab")
 			(effects
@@
 		)
 		(fp_line
+			(start 0.625 -1.04)
+			(end 0.625 -0.24)
+			(stroke
+				(width 0.05)
+				(type solid)
+			)
+			(layer "F.Fab")
+		)
+		(fp_line
 			(start -0.645 -1.04)
 			(end -0.645 -0.24)
@@
 		)
 		(fp_line
+			(start 1.025 -0.64)
+			(end 0.225 -0.64)
+			(stroke
+				(width 0.05)
+				(type solid)
+			)
+			(layer "F.Fab")
+		)
+		(fp_line
+			(start -0.245 -0.64)
+			(end -1.045 -0.64)
+			(stroke
+				(width 0.05)
+				(type solid)
+			)
+			(layer "F.Fab")
+		)
+		(fp_line
+			(start 0.625 0.23)
+			(end 0.625 1.03)
+			(stroke
+				(width 0.05)
+				(type solid)
+			)
+			(layer "F.Fab")
+		)
+		(fp_line
 			(start -0.645 0.23)
 			(end -0.645 1.03)
@@
 		)
 		(fp_line
+			(start 1.025 0.63)
+			(end 0.225 0.63)
+			(stroke
+				(width 0.05)
+				(type solid)
+			)
+			(layer "F.Fab")
+		)
+		(fp_line
+			(start -0.245 0.63)
+			(end -1.045 0.63)
+			(stroke
+				(width 0.05)
+				(type solid)
+			)
+			(layer "F.Fab")
+		)
+		(fp_line
+			(start 0.625 1.5)
+			(end 0.625 2.3)
+			(stroke
+				(width 0.05)
+				(type solid)
+			)
+			(layer "F.Fab")
+		)
+		(fp_line
 			(start -0.645 1.5)
 			(end -0.645 2.3)
@@
 		)
 		(fp_line
-			(start -0.245 -0.64)
-			(end -1.045 -0.64)
-			(stroke
-				(width 0.05)
-				(type solid)
-			)
-			(layer "F.Fab")
-		)
-		(fp_line
-			(start -0.245 0.63)
-			(end -1.045 0.63)
+			(start 1.025 1.9)
+			(end 0.225 1.9)
 			(stroke
 				(width 0.05)
@@
 			(layer "F.Fab")
 		)
-		(fp_line
-			(start 0.625 -1.04)
-			(end 0.625 -0.24)
-			(stroke
-				(width 0.05)
-				(type solid)
-			)
-			(layer "F.Fab")
-		)
-		(fp_line
-			(start 0.625 0.23)
-			(end 0.625 1.03)
-			(stroke
-				(width 0.05)
-				(type solid)
-			)
-			(layer "F.Fab")
-		)
-		(fp_line
-			(start 0.625 1.5)
-			(end 0.625 2.3)
-			(stroke
-				(width 0.05)
-				(type solid)
-			)
-			(layer "F.Fab")
-		)
-		(fp_line
-			(start 1.025 -0.64)
-			(end 0.225 -0.64)
-			(stroke
-				(width 0.05)
-				(type solid)
-			)
-			(layer "F.Fab")
-		)
-		(fp_line
-			(start 1.025 0.63)
-			(end 0.225 0.63)
-			(stroke
-				(width 0.05)
-				(type solid)
-			)
-			(layer "F.Fab")
-		)
-		(fp_line
-			(start 1.025 1.9)
-			(end 0.225 1.9)
-			(stroke
-				(width 0.05)
-				(type solid)
-			)
-			(layer "F.Fab")
-		)
-		(pad "" np_thru_hole circle
-			(at -2.55 -1.91 270)
+		(pad "" np_thru_hole circle
+			(at -2.55 -1.91)
 			(size 2.3749 2.3749)
 			(drill 2.3749)
@@
 		)
 		(pad "" np_thru_hole circle
-			(at -2.55 1.265 270)
+			(at -2.55 1.265)
 			(size 2.3749 2.3749)
 			(drill 2.3749)
@@
 		)
 		(pad "" np_thru_hole circle
-			(at -1.026 3.17 270)
+			(at -1.026 3.17)
 			(size 0.9906 0.9906)
 			(drill 0.9906)
@@
 		)
 		(pad "" np_thru_hole circle
-			(at -0.01 -1.91 270)
+			(at -0.01 -1.91)
 			(size 0.9906 0.9906)
 			(drill 0.9906)
@@
 		)
 		(pad "" np_thru_hole circle
-			(at 1.006 3.17 270)
+			(at 1.006 3.17)
 			(size 0.9906 0.9906)
 			(drill 0.9906)
@@
 		)
 		(pad "" np_thru_hole circle
-			(at 2.53 -1.91 270)
+			(at 2.53 -1.91)
 			(size 2.3749 2.3749)
 			(drill 2.3749)
@@
 		)
 		(pad "" np_thru_hole circle
-			(at 2.53 1.265 270)
+			(at 2.53 1.265)
 			(size 2.3749 2.3749)
 			(drill 2.3749)
@@
 		)
 		(pad "1" smd roundrect
-			(at -3.5 5.5)
+			(at -3.5 5.5 90)
 			(size 1.2 3)
 			(layers "F.Cu" "F.Mask")
@@
 		)
 		(pad "1" smd roundrect
-			(at -3.375 13.5)
+			(at -3.375 13.5 90)
 			(size 0.9 8)
 			(layers "F.Cu" "F.Mask")
@@
 		)
 		(pad "1" thru_hole circle
-			(at -0.645 -0.64 270)
+			(at -0.645 -0.64)
 			(size 1 1)
 			(drill 0.65)
@@
 		)
 		(pad "2" smd roundrect
-			(at -2.025 13.5)
+			(at -2.025 13.5 90)
 			(size 0.9 8)
 			(layers "F.Cu" "F.Mask")
@@
 		)
 		(pad "2" thru_hole circle
-			(at 0.625 -0.64 270)
+			(at 0.625 -0.64)
 			(size 1 1)
 			(drill 0.65)
@@
 		)
 		(pad "3" smd roundrect
-			(at -0.675 13.5)
+			(at -0.675 13.5 90)
 			(size 0.9 8)
 			(layers "F.Cu" "F.Mask")
@@
 		)
 		(pad "3" thru_hole circle
-			(at -0.645 0.63 270)
+			(at -0.645 0.63)
 			(size 1 1)
 			(drill 0.65)
@@
 		)
 		(pad "4" thru_hole circle
-			(at 0.625 0.63 270)
+			(at 0.625 0.63)
 			(size 1 1)
 			(drill 0.65)
@@
 		)
 		(pad "4" smd roundrect
-			(at 0.675 13.5)
+			(at 0.675 13.5 90)
 			(size 0.9 8)
 			(layers "F.Cu" "F.Mask")
@@
 		)
 		(pad "5" thru_hole circle
-			(at -0.645 1.9 270)
+			(at -0.645 1.9)
 			(size 1 1)
 			(drill 0.65)
@@
 		)
 		(pad "5" smd roundrect
-			(at 2.025 13.5)
+			(at 2.025 13.5 90)
 			(size 0.9 8)
 			(layers "F.Cu" "F.Mask")
@@
 		)
 		(pad "5" smd roundrect
-			(at 3.5 5.5)
+			(at 3.5 5.5 90)
 			(size 1.2 3)
 			(layers "F.Cu" "F.Mask")
@@
 		)
 		(pad "6" thru_hole circle
-			(at 0.625 1.9 270)
+			(at 0.625 1.9)
 			(size 1 1)
 			(drill 0.65)
@@
 		)
 		(pad "6" smd roundrect
-			(at 3.375 13.5)
-			(size 0.9 8)
-			(layers "F.Cu" "F.Mask")
+			(at 3.375 13.5 90)
+			(size 0.9 8)
+			(layers "F.Cu" "F.Mask")

Commit message: feat: jtag connector/programer rename
Parts:
- moved JTAG 32.4 mm to (44.0, 97.0), turned to 180 degrees
Changed lines of the file:
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@@
 	(footprint "Woki:CONN_TC2030_JTAG_PROBE"
 		(layer "F.Cu")
-		(at 60.08 68.974 90)
+		(at 43.975 97.05 180)
 		(descr "Generated from CONN_TC2030_JTAG.kicad_mod; TC2030 pitch 1.27 mm, C5157236 tip 0.80 mm leaves 0.47 mm between tips, barrel 1.20 mm leaves 0.07 mm between barrels")
 		(tags "tc2030 jtag swd pogo probe card-edge")
 		(property "Reference" "JTAG"
-			(at 0 6.875 90)
+			(at 0 6.875 0)
 			(layer "F.SilkS")
 			(effects
@@
 			)
 		)
+		(property "Value" "CONN_TC2030_JTAG"
+			(at 0 20 0)
+			(layer "F.Fab")
+			(effects
+				(font
+					(size 1 1)
+					(thickness 0.15)
+				)
+			)
+		)
 		(property "Datasheet" "https://www.tag-connect.com/wp-content/uploads/bsk-pdf-manager/TC2030-CTX_1.pdf"
-			(at 0 0 90)
+			(at 0 0 0)
 			(layer "F.Fab")
 			(hide yes)
@@
 		)
 		(property "Description" "Tag-Connect ARM Cortex SWD JTAG connector, 6 pin"
-			(at 0 0 90)
+			(at 0 0 0)
 			(layer "F.Fab")
 			(hide yes)
-			(effects
-				(font
-					(size 1 1)
-					(thickness 0.15)
-				)
-			)
-		)
-		(property "Value" "CONN_TC2030_JTAG"
-			(at 0 20 90)
-			(layer "F.Fab")
 			(effects
 				(font
@@
 		)
 		(fp_line
+			(start 1.025 1.9)
+			(end 0.225 1.9)
+			(stroke
+				(width 0.05)
+				(type solid)
+			)
+			(layer "F.Fab")
+		)
+		(fp_line
+			(start 1.025 0.63)
+			(end 0.225 0.63)
+			(stroke
+				(width 0.05)
+				(type solid)
+			)
+			(layer "F.Fab")
+		)
+		(fp_line
+			(start 1.025 -0.64)
+			(end 0.225 -0.64)
+			(stroke
+				(width 0.05)
+				(type solid)
+			)
+			(layer "F.Fab")
+		)
+		(fp_line
+			(start 0.625 1.5)
+			(end 0.625 2.3)
+			(stroke
+				(width 0.05)
+				(type solid)
+			)
+			(layer "F.Fab")
+		)
+		(fp_line
+			(start 0.625 0.23)
+			(end 0.625 1.03)
+			(stroke
+				(width 0.05)
+				(type solid)
+			)
+			(layer "F.Fab")
+		)
+		(fp_line
 			(start 0.625 -1.04)
 			(end 0.625 -0.24)
@@
 		)
 		(fp_line
+			(start -0.245 1.9)
+			(end -1.045 1.9)
+			(stroke
+				(width 0.05)
+				(type solid)
+			)
+			(layer "F.Fab")
+		)
+		(fp_line
+			(start -0.245 0.63)
+			(end -1.045 0.63)
+			(stroke
+				(width 0.05)
+				(type solid)
+			)
+			(layer "F.Fab")
+		)
+		(fp_line
+			(start -0.245 -0.64)
+			(end -1.045 -0.64)
+			(stroke
+				(width 0.05)
+				(type solid)
+			)
+			(layer "F.Fab")
+		)
+		(fp_line
+			(start -0.645 1.5)
+			(end -0.645 2.3)
+			(stroke
+				(width 0.05)
+				(type solid)
+			)
+			(layer "F.Fab")
+		)
+		(fp_line
+			(start -0.645 0.23)
+			(end -0.645 1.03)
+			(stroke
+				(width 0.05)
+				(type solid)
+			)
+			(layer "F.Fab")
+		)
+		(fp_line
 			(start -0.645 -1.04)
 			(end -0.645 -0.24)
@@
 			(layer "F.Fab")
 		)
-		(fp_line
-			(start 1.025 -0.64)
-			(end 0.225 -0.64)
-			(stroke
-				(width 0.05)
-				(type solid)
-			)
-			(layer "F.Fab")
-		)
-		(fp_line
-			(start -0.245 -0.64)
-			(end -1.045 -0.64)
-			(stroke
-				(width 0.05)
-				(type solid)
-			)
-			(layer "F.Fab")
-		)
-		(fp_line
-			(start 0.625 0.23)
-			(end 0.625 1.03)
-			(stroke
-				(width 0.05)
-				(type solid)
-			)
-			(layer "F.Fab")
-		)
-		(fp_line
-			(start -0.645 0.23)
-			(end -0.645 1.03)
-			(stroke
-				(width 0.05)
-				(type solid)
-			)
-			(layer "F.Fab")
-		)
-		(fp_line
-			(start 1.025 0.63)
-			(end 0.225 0.63)
-			(stroke
-				(width 0.05)
-				(type solid)
-			)
-			(layer "F.Fab")
-		)
-		(fp_line
-			(start -0.245 0.63)
-			(end -1.045 0.63)
-			(stroke
-				(width 0.05)
-				(type solid)
-			)
-			(layer "F.Fab")
-		)
-		(fp_line
-			(start 0.625 1.5)
-			(end 0.625 2.3)
-			(stroke
-				(width 0.05)
-				(type solid)
-			)
-			(layer "F.Fab")
-		)
-		(fp_line
-			(start -0.645 1.5)
-			(end -0.645 2.3)
-			(stroke
-				(width 0.05)
-				(type solid)
-			)
-			(layer "F.Fab")
-		)
-		(fp_line
-			(start 1.025 1.9)
-			(end 0.225 1.9)
-			(stroke
-				(width 0.05)
-				(type solid)
-			)
-			(layer "F.Fab")
-		)
-		(fp_line
-			(start -0.245 1.9)
-			(end -1.045 1.9)
-			(stroke
-				(width 0.05)
-				(type solid)
-			)
-			(layer "F.Fab")
-		)
-		(pad "" np_thru_hole circle
-			(at -2.55 -1.91)
+		(pad "" np_thru_hole circle
+			(at -2.55 -1.91 90)
 			(size 2.3749 2.3749)
 			(drill 2.3749)
@@
 		)
 		(pad "" np_thru_hole circle
-			(at -2.55 1.265)
+			(at -2.55 1.265 90)
 			(size 2.3749 2.3749)
 			(drill 2.3749)
@@
 		)
 		(pad "" np_thru_hole circle
-			(at -1.026 3.17)
+			(at -1.026 3.17 90)
 			(size 0.9906 0.9906)
 			(drill 0.9906)
@@
 		)
 		(pad "" np_thru_hole circle
-			(at -0.01 -1.91)
+			(at -0.01 -1.91 90)
 			(size 0.9906 0.9906)
 			(drill 0.9906)
@@
 		)
 		(pad "" np_thru_hole circle
-			(at 1.006 3.17)
+			(at 1.006 3.17 90)
 			(size 0.9906 0.9906)
 			(drill 0.9906)
@@
 		)
 		(pad "" np_thru_hole circle
-			(at 2.53 -1.91)
+			(at 2.53 -1.91 90)
 			(size 2.3749 2.3749)
 			(drill 2.3749)
@@
 		)
 		(pad "" np_thru_hole circle
-			(at 2.53 1.265)
+			(at 2.53 1.265 90)
 			(size 2.3749 2.3749)
 			(drill 2.3749)
@@
 		)
 		(pad "1" smd roundrect
-			(at -3.5 5.5 90)
+			(at -3.5 5.5 180)
 			(size 1.2 3)
 			(layers "F.Cu" "F.Mask")
@@
 		)
 		(pad "1" smd roundrect
-			(at -3.375 13.5 90)
+			(at -3.375 13.5 180)
 			(size 0.9 8)
 			(layers "F.Cu" "F.Mask")
@@
 		)
 		(pad "1" thru_hole circle
-			(at -0.645 -0.64)
+			(at -0.645 -0.64 90)
 			(size 1 1)
 			(drill 0.65)
@@
 		)
 		(pad "2" smd roundrect
-			(at -2.025 13.5 90)
+			(at -2.025 13.5 180)
 			(size 0.9 8)
 			(layers "F.Cu" "F.Mask")
@@
 		)
 		(pad "2" thru_hole circle
-			(at 0.625 -0.64)
+			(at 0.625 -0.64 90)
 			(size 1 1)
 			(drill 0.65)
@@
 		)
 		(pad "3" smd roundrect
-			(at -0.675 13.5 90)
+			(at -0.675 13.5 180)
 			(size 0.9 8)
 			(layers "F.Cu" "F.Mask")
@@
 		)
 		(pad "3" thru_hole circle
-			(at -0.645 0.63)
+			(at -0.645 0.63 90)
 			(size 1 1)
 			(drill 0.65)
@@
 		)
 		(pad "4" thru_hole circle
-			(at 0.625 0.63)
+			(at 0.625 0.63 90)
 			(size 1 1)
 			(drill 0.65)
@@
 		)
 		(pad "4" smd roundrect
-			(at 0.675 13.5 90)
+			(at 0.675 13.5 180)
 			(size 0.9 8)
 			(layers "F.Cu" "F.Mask")
@@
 		)
 		(pad "5" thru_hole circle
-			(at -0.645 1.9)
+			(at -0.645 1.9 90)
 			(size 1 1)
 			(drill 0.65)
@@
 		)
 		(pad "5" smd roundrect
-			(at 2.025 13.5 90)
+			(at 2.025 13.5 180)
 			(size 0.9 8)
 			(layers "F.Cu" "F.Mask")
@@
 		)
 		(pad "5" smd roundrect
-			(at 3.5 5.5 90)
+			(at 3.5 5.5 180)
 			(size 1.2 3)
 			(layers "F.Cu" "F.Mask")
@@
 		)
 		(pad "6" thru_hole circle
-			(at 0.625 1.9)
+			(at 0.625 1.9 90)
 			(size 1 1)
 			(drill 0.65)
@@
 		)
 		(pad "6" smd roundrect
-			(at 3.375 13.5 90)
-			(size 0.9 8)
-			(layers "F.Cu" "F.Mask")
+			(at 3.375 13.5 180)
+			(size 0.9 8)
+			(layers "F.Cu" "F.Mask")

Commit message: feat: outline
Parts:
- moved JTAG 1.22 mm to (43.0, 96.2)
Other:
- board size 50 x 50 mm -> 61.2 x 50 mm
Changed lines of the file:
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@@
 	)
 	(footprint "Woki:CONN_TC2030_JTAG_PROBE"
+		(locked yes)
 		(layer "F.Cu")
-		(at 43.975 97.05 180)
+		(at 43.05 96.25 180)
 		(descr "Generated from CONN_TC2030_JTAG.kicad_mod; TC2030 pitch 1.27 mm, C5157236 tip 0.80 mm leaves 0.47 mm between tips, barrel 1.20 mm leaves 0.07 mm between barrels")
 		(tags "tc2030 jtag swd pogo probe card-edge")
@@
 		(layer "F.SilkS")
 	)
+	(gr_rect
+		(start 38.8 78.75)
+		(end 47.3 100)
+		(radius 1)
+		(stroke
+			(width 0.1)
+			(type default)
+		)
+		(fill no)
+		(layer "Edge.Cuts")
+	)
+	(gr_line
+		(start 47.3 81.1)
+		(end 50 81.1)
+		(stroke
+			(width 0.1)
+			(type default)
+		)
+		(layer "Edge.Cuts")
+	)
+	(gr_rect
+		(start 47.3 81.1)
+		(end 50 84.1)
+		(stroke
+			(width 0.1)
+			(type default)
+		)
+		(fill no)
+		(layer "Edge.Cuts")
+	)
+	(gr_line
+		(start 47.3 84.1)
+		(end 50 84.1)
+		(stroke
+			(width 0.1)
+			(type default)
+		)
+		(layer "Edge.Cuts")
+	)
+	(gr_line
+		(start 47.3 93.6)
+		(end 50 93.6)
+		(stroke
+			(width 0.1)
+			(type default)
+		)
+		(layer "Edge.Cuts")
+	)
+	(gr_rect
+		(start 47.3 93.6)
+		(end 50 96.6)
+		(stroke
+			(width 0.1)
+			(type default)
+		)
+		(fill no)
+		(layer "Edge.Cuts")
+	)
+	(gr_line
+		(start 47.3 96.6)
+		(end 50 96.6)
+		(stroke
+			(width 0.1)
+			(type default)
+		)
+		(layer "Edge.Cuts")
+	)
 	(gr_line

Commit message: feat: break vias
Routing:
- net unconnected-(J5-VCC-Pad1): track 0.00 -> 8.05 mm
- net +12V_BULK: vias 0 -> 2
- net (no net): vias 0 -> 14
Other:
- outline, holes or cut-outs redrawn
