File: boards/01-power/stm32.kicad_sch (KiCad schematic)
At the start: 26 parts, among them J3 TC2030, SW1 SW_BOOT, SW2 SW_BOOT, SW3 SW_BOOT, U3 STM32F405RGTx, Y1 16Mhz

Commit message: wip: 3.3v
Connections:
- net GND: now also R5.2, R6.2; no longer D1.1 (K), D2.1 (K)
- net LED_ERROR: now also D2.2 (A); no longer R6.1
- net LED_STATUS: now also D1.2 (A); no longer R5.1
- new net: D1.1 (K), R5.1
- new net: D2.1 (K), R6.1
Other:
- moved on the sheet: D1, D2

Commit message: wip: buck (plan layout rough)
Parts:
- removed R8: 10k, Resistor_SMD:R_0603_1608Metric, symbol Device:R_Small
- removed SW3: SW_BOOT, Woki:SW_B3U_1000P, symbol Switch:SW_Push
Connections:
- net USR_BTN2: no longer names the net of U3.11 (PC3)

Commit message: wip: stm
Connections:
- net LED_ERROR: now also U3.25 (PC5); no longer U3.3 (PC14)
- net LED_STATUS: now also U3.24 (PC4); no longer U3.2 (PC13)
Changed lines of the file:
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@@
-	(wire
-		(pts
-			(xy 127 101.6) (xy 128.27 101.6)
-		)
-		(stroke
-			(width 0)
-			(type default)
-		)
-	)
 	(wire
 		(pts
@@
 	(wire
 		(pts
+			(xy 127 78.74) (xy 128.27 78.74)
+		)
+		(stroke
+			(width 0)
+			(type default)
+		)
+	)
+	(wire
+		(pts
 			(xy 127 73.66) (xy 128.27 73.66)
 		)
@@
 	(wire
 		(pts
+			(xy 127 81.28) (xy 128.27 81.28)
+		)
+		(stroke
+			(width 0)
+			(type default)
+		)
+	)
+	(wire
+		(pts
 			(xy 87.63 72.39) (xy 87.63 66.04)
 		)
@@
 	(wire
 		(pts
-			(xy 127 104.14) (xy 128.27 104.14)
-		)
-		(stroke
-			(width 0)
-			(type default)
-		)
-	)
-	(wire
-		(pts
 			(xy 127 25.4) (xy 134.62 25.4)
 		)
@@
 			(width 0)
 			(type default)
-		)
-	)
-	(label "LED_STATUS"
-		(at 127 101.6 180)
-		(effects
-			(font
-				(size 1.27 1.27)
-			)
-			(justify right bottom)
-		)
-	)
-	(label "LED_ERROR"
-		(at 127 104.14 180)
-		(effects
-			(font
-				(size 1.27 1.27)
-			)
-			(justify right bottom)
 		)
 	)
@@
 		)
 	)
+	(label "LED_ERROR"
+		(at 127 81.28 180)
+		(effects
+			(font
+				(size 1.27 1.27)
+			)
+			(justify right bottom)
+		)
+	)
 	(label "~{STM_RESET}"
 		(at 107.95 43.18 180)
@@
 		)
 	)
+	(label "LED_STATUS"
+		(at 127 78.74 180)
+		(effects
+			(font
+				(size 1.27 1.27)
+			)
+			(justify right bottom)
+		)
+	)

Commit message: finish: stm32/added icons
Parts:
- removed R4: 10k, Resistor_SMD:R_0603_1608Metric, symbol Device:R_Small
- removed SW1: SW_BOOT, Woki:SW_B3U_1000P, symbol Switch:SW_Push

Commit message: poe: class 8 negotiate(max around 62W-71W at PD)
Parts:
- added R8: 10k, Resistor_SMD:R_0603_1608Metric, symbol Device:R_Small
Connections:
- net BOOT0: now also R8.1
- net GND: now also R8.2
Changed lines of the file:
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@@
+	(wire
+		(pts
+			(xy 25.4 35.56) (xy 25.4 36.83)
+		)
+		(stroke
+			(width 0)
+			(type default)
+		)
+	)
 	(wire
 		(pts
@@
 		(pts
 			(xy 127 81.28) (xy 128.27 81.28)
+		)
+		(stroke
+			(width 0)
+			(type default)
+		)
+	)
+	(wire
+		(pts
+			(xy 25.4 41.91) (xy 25.4 44.45)
 		)
 		(stroke
@@
 			)
 			(justify left bottom)
+		)
+	)
+	(label "BOOT0"
+		(at 25.4 35.56 180)
+		(effects
+			(font
+				(size 1.27 1.27)
+			)
+			(justify right bottom)
 		)
 	)
@@
 	)
 	(symbol
+		(lib_id "power:GND")
+		(at 25.4 44.45 0)
+		(unit 1)
+		(body_style 1)
+		(exclude_from_sim no)
+		(in_bom yes)
+		(on_board yes)
+		(in_pos_files yes)
+		(dnp no)
+		(fields_autoplaced yes)
+		(property "Reference" "#PWR017"
+			(at 25.4 50.8 0)
+			(hide yes)
+			(show_name no)
+			(do_not_autoplace no)
+			(effects
+				(font
+					(size 1.27 1.27)
+				)
+			)
+		)
+		(property "Value" "GND"
+			(at 25.4 49.53 0)
+			(show_name no)
+			(do_not_autoplace no)
+			(effects
+				(font
+					(size 1.27 1.27)
+				)
+			)
+		)
+		(property "Footprint" ""
+			(at 25.4 44.45 0)
+			(hide yes)
+			(show_name no)
+			(do_not_autoplace no)
+			(effects
+				(font
+					(size 1.27 1.27)
+				)
+			)
+		)
+		(property "Datasheet" ""
+			(at 25.4 44.45 0)
+			(hide yes)
+			(show_name no)
+			(do_not_autoplace no)
+			(effects
+				(font
+					(size 1.27 1.27)
+				)
+			)
+		)
+		(property "Description" "Power symbol creates a global label with name \"GND\" , ground"
+			(at 25.4 44.45 0)
+			(hide yes)
+			(show_name no)
+			(do_not_autoplace no)
+			(effects
+				(font
+					(size 1.27 1.27)
+				)
+			)
+		)
+		(pin "1"
+		)
+		(instances
+			(project "power"
+				(path "/de291139-592d-56bb-a3cc-5961c2880226/c70ce39d-69a4-460d-bc53-bac390a88578"
+					(reference "#PWR017")
+					(unit 1)
+				)
+			)
+		)
+	)
+	(symbol
 		(lib_id "Switch:SW_Push")
 		(at 39.37 29.21 90)
@@
 					(unit 1)
 				)
+			)
+		)
+	)
+	(symbol
+		(lib_id "Device:R_Small")
+		(at 25.4 39.37 0)
+		(unit 1)
+		(body_style 1)
+		(exclude_from_sim no)
+		(in_bom yes)
+		(on_board yes)
+		(in_pos_files yes)
+		(dnp no)
+		(property "Reference" "R8"
+			(at 26.67 38.1 0)
+			(show_name no)
+			(do_not_autoplace no)
+			(effects
+				(font
+					(size 1.016 1.016)
+				)
+				(justify left)
+			)
+		)
+		(property "Value" "10k"
+			(at 26.416 40.64 0)
+			(show_name no)
+			(do_not_autoplace no)
+			(effects
+				(font
+					(size 1.27 1.27)
+				)
+				(justify left)
+			)
+		)
+		(property "Footprint" "Resistor_SMD:R_0603_1608Metric"
+			(at 25.4 39.37 0)
+			(hide yes)
+			(show_name no)
+			(do_not_autoplace no)
+			(effects
+				(font
+					(size 1.27 1.27)
+				)
+			)
+		)
+		(property "Datasheet" ""
+			(at 25.4 39.37 0)
+			(hide yes)
+			(show_name no)
+			(do_not_autoplace no)
+			(effects
+				(font
+					(size 1.27 1.27)
+				)
+			)
+		)
+		(property "Description" "Resistor, small symbol"
+			(at 25.4 39.37 0)
+			(hide yes)
+			(show_name no)
+			(do_not_autoplace no)
+			(effects
+				(font
+					(size 1.27 1.27)
+				)
+			)
+		)
+		(pin "2"
+		)
+		(pin "1"
+		)
+		(instances
+			(project "power"
+				(path "/de291139-592d-56bb-a3cc-5961c2880226/c70ce39d-69a4-460d-bc53-bac390a88578"
+					(reference "R8")
+					(unit 1)
+				)
