File: boards/02-fpga-control/fpga_control.kicad_pcb (KiCad board)
At the start: 6 copper layers, 50 x 50 mm, 6 parts, among them J1 CONN_DF40_100P_M, J2 CONN_DF40_100P_F

Commit message: wip: 8 layer stackup
Other:
- copper layers 6 -> 8
Changed lines of the file:
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@@
 		(8 "In3.Cu" power "PWR")
 		(10 "In4.Cu" power "GND2")
+		(12 "In5.Cu" signal "SIG3")
+		(14 "In6.Cu" power "GND3")
 		(2 "B.Cu" signal)
 		(5 "F.SilkS" user "F.Silkscreen")
@@
 				(type "core")
 				(color "#FF9B30FF")
-				(thickness 0.545)
+				(thickness 0.18)
 				(material "FR4")
 				(epsilon_r 4.5)
@@
 				(type "core")
 				(color "#FF7030FF")
-				(thickness 0.545)
+				(thickness 0.56)
 				(material "FR4")
 				(epsilon_r 4.5)
@@
 				(thickness 0.1)
 				(material "FR4")
+				(epsilon_r 4.5)
+				(loss_tangent 0.02)
+			)
+			(layer "In5.Cu"
+				(type "copper")
+				(thickness 0.035)
+			)
+			(layer "dielectric 6"
+				(type "core")
+				(color "#FF9B30FF")
+				(thickness 0.18)
+				(material "FR4")
+				(epsilon_r 4.5)
+				(loss_tangent 0.02)
+			)
+			(layer "In6.Cu"
+				(type "copper")
+				(thickness 0.035)
+			)
+			(layer "dielectric 7"
+				(type "prepreg")
+				(color "#30FF19FF")
+				(thickness 0.1)
+				(material "FR4")
